File: hardware/ziffy_board_v6.brd (EAGLE design)
At the start: 52 x 50 mm, 28 parts, among them IC1 74HC125, IC2 74HC125, IC3 74HC125, IC4 74HC125, IC5 74HC125, IC6 74HC125

Commit message: trying all the angles (ba-dum-tish)
Parts:
- R1, R2, R3: device A_butts:R0805 -> A_butts:RESISTOR-AXIAL-PTH-5.08MM
- moved BUSY 9.00 mm to (37.5, 46.5)
- moved R3 8.71 mm to (46.2, 42.3), turned to 225 degrees
- moved HI! 8.60 mm to (46.1, 46.5)
- moved R1 8.51 mm to (38.0, 42.3), turned to 225 degrees
- moved R2 0.32 mm to (42.1, 42.3), turned to 225 degrees
- moved ERR 0.20 mm to (41.8, 46.5)
Connections:
- net GND: now also R1.P$2, R2.P$2, R3.P$2; no longer R1.2, R2.2, R3.2
- net N$1: now also R1.P$1; no longer R1.1
- net N$2: now also R2.P$1; no longer R2.1
- net N$3: now also R3.P$1; no longer R3.1
Routing:
- net BUSY: track 67.8 -> 56.3 mm, vias 0 -> 1
- net HELLO: track 50.6 -> 59.7 mm
Changed lines of the file:
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@@
 <elements>
 <element name="C1" library="A_butts" package="C025-024X044" value="0.1uF" x="16" y="44.27" rot="R90"/>
-<element name="BUSY" library="A_butts" package="LED3MM" value="YELLOW" x="46.5" y="46.5" smashed="yes" rot="R270">
-<attribute name="NAME" x="46.5" y="48.843" size="0.8" layer="25" font="vector" ratio="12" rot="SR180" align="top-center"/>
-</element>
-<element name="ERR" library="A_butts" package="LED3MM" value="RED" x="42" y="46.5" smashed="yes" rot="R270">
-<attribute name="NAME" x="42" y="48.843" size="0.8" layer="25" font="vector" ratio="12" rot="SR180" align="top-center"/>
-</element>
-<element name="HI!" library="A_butts" package="LED3MM" value="GREEN" x="37.5" y="46.5" smashed="yes" rot="R270">
-<attribute name="NAME" x="37.5" y="48.843" size="0.8" layer="25" font="vector" ratio="12" rot="SR180" align="top-center"/>
+<element name="BUSY" library="A_butts" package="LED3MM" value="YELLOW" x="37.5" y="46.5" smashed="yes" rot="R270">
+<attribute name="NAME" x="37.5" y="48.8" size="0.8" layer="25" font="vector" ratio="12" rot="SR180" align="top-center"/>
+</element>
+<element name="ERR" library="A_butts" package="LED3MM" value="RED" x="41.8" y="46.5" smashed="yes" rot="R270">
+<attribute name="NAME" x="41.8" y="48.8" size="0.8" layer="25" font="vector" ratio="12" rot="SR180" align="top-center"/>
+</element>
+<element name="HI!" library="A_butts" package="LED3MM" value="GREEN" x="46.1" y="46.5" smashed="yes" rot="R270">
+<attribute name="NAME" x="46.076090625" y="48.802940625" size="0.8" layer="25" font="vector" ratio="12" rot="SR180" align="top-center"/>
 </element>
 <element name="R4" library="A_butts" package="RESISTOR-AXIAL-PTH-5.08MM" value="10k" x="47" y="17" rot="R90"/>
@@
 <element name="C3" library="A_butts" package="C025-024X044" value="0.1uF" x="16" y="25.5" rot="R90"/>
 <element name="C4" library="A_butts" package="C025-024X044" value="0.1uF" x="16" y="13.97" rot="R90"/>
-<element name="R1" library="A_butts" package="R0805" value="330R" x="46.5" y="42" rot="R270"/>
-<element name="R2" library="A_butts" package="R0805" value="330R" x="42" y="42" rot="R270"/>
-<element name="R3" library="A_butts" package="R0805" value="330R" x="37.5" y="42" rot="R270"/>
+<element name="R1" library="A_butts" package="RESISTOR-AXIAL-PTH-5.08MM" value="330R" x="38" y="42.3" smashed="yes" rot="R225">
+<attribute name="NAME" x="37.51446875" y="42.71446875" size="0.4064" layer="25" font="vector" ratio="12" rot="R45" align="bottom-center"/>
+<attribute name="VALUE" x="38.485528125" y="41.785528125" size="0.4064" layer="27" font="vector" ratio="12" rot="R45" align="top-center"/>
+</element>
+<element name="R2" library="A_butts" package="RESISTOR-AXIAL-PTH-5.08MM" value="330R" x="42.1" y="42.3" smashed="yes" rot="R225">
+<attribute name="NAME" x="41.68553125" y="42.81446875" size="0.4064" layer="25" font="vector" ratio="12" rot="R45" align="bottom-center"/>
+<attribute name="VALUE" x="42.585528125" y="41.785528125" size="0.4064" layer="27" font="vector" ratio="12" rot="R45" align="top-center"/>
+</element>
+<element name="R3" library="A_butts" package="RESISTOR-AXIAL-PTH-5.08MM" value="330R" x="46.2" y="42.3" smashed="yes" rot="R225">
+<attribute name="NAME" x="45.78553125" y="42.81446875" size="0.4064" layer="25" font="vector" ratio="12" rot="R45" align="bottom-center"/>
+<attribute name="VALUE" x="46.685528125" y="41.785528125" size="0.4064" layer="27" font="vector" ratio="12" rot="R45" align="top-center"/>
+</element>
 <element name="TARGET_RESET" library="A_butts" package="DTS-6-SMALL-PADS" value="SPST-NO-TACT6MM-PTH-SMALL-PADS" x="40" y="5" rot="R90"/>
 <element name="IC1" library="A_butts" package="SO14" value="74HC125" x="10" y="45.5" smashed="yes" rot="R180">
@@
 <contactref element="C1" pad="2"/>
 <contactref element="C2" pad="2"/>
-<contactref element="R1" pad="2"/>
-<contactref element="R2" pad="2"/>
-<contactref element="R3" pad="2"/>
+<contactref element="R1" pad="P$2"/>
+<contactref element="R2" pad="P$2"/>
+<contactref element="R3" pad="P$2"/>
 <contactref element="SHIELD" pad="GND@1"/>
 <contactref element="SHIELD" pad="GND@0"/>
@@
 <wire x1="3.5" y1="32.05" x2="3.5" y2="44.7" width="0.2" layer="16"/>
 <wire x1="3.5" y1="44.7" x2="7.2" y2="48.4" width="0.2" layer="16"/>
-<wire x1="7.2" y1="48.4" x2="36.87" y2="48.4" width="0.2" layer="16"/>
-<wire x1="36.87" y1="48.4" x2="37.5" y2="47.77" width="0.2" layer="16"/>
+<wire x1="7.2" y1="48.4" x2="35.4" y2="48.4" width="0.2" layer="16"/>
+<wire x1="35.4" y1="48.4" x2="36" y2="49" width="0.2" layer="16"/>
+<wire x1="36" y1="49" x2="44.87" y2="49" width="0.2" layer="16"/>
+<wire x1="44.87" y1="49" x2="46.1" y2="47.77" width="0.2" layer="16"/>
 </signal>
 <signal name="ERROR">
@@
 <wire x1="3.9" y1="28.64" x2="3.9" y2="44.6" width="0.2" layer="16"/>
 <wire x1="3.9" y1="44.6" x2="7.3" y2="48" width="0.2" layer="16"/>
-<wire x1="7.3" y1="48" x2="34.5" y2="48" width="0.2" layer="16"/>
-<wire x1="34.5" y1="48" x2="36" y2="46.5" width="0.2" layer="16"/>
-<wire x1="36" y1="46.5" x2="40.73" y2="46.5" width="0.2" layer="16"/>
-<wire x1="40.73" y1="46.5" x2="42" y2="47.77" width="0.2" layer="16"/>
+<wire x1="7.3" y1="48" x2="35" y2="48" width="0.2" layer="16"/>
+<wire x1="35" y1="48" x2="36.5" y2="46.5" width="0.2" layer="16"/>
+<wire x1="36.5" y1="46.5" x2="40.53" y2="46.5" width="0.2" layer="16"/>
+<wire x1="40.53" y1="46.5" x2="41.8" y2="47.77" width="0.2" layer="16"/>
 </signal>
 <signal name="BUSY">
@@
 <wire x1="4.3" y1="26.5" x2="4.3" y2="44.5" width="0.2" layer="16"/>
 <wire x1="4.3" y1="44.5" x2="7.4" y2="47.6" width="0.2" layer="16"/>
-<wire x1="7.4" y1="47.6" x2="32.9" y2="47.6" width="0.2" layer="16"/>
-<wire x1="32.9" y1="47.6" x2="36.5" y2="44" width="0.2" layer="16"/>
-<wire x1="36.5" y1="44" x2="42.73" y2="44" width="0.2" layer="16"/>
-<wire x1="42.73" y1="44" x2="46.5" y2="47.77" width="0.2" layer="16"/>
+<wire x1="7.4" y1="47.6" x2="31.9" y2="47.6" width="0.2" layer="16"/>
+<wire x1="31.9" y1="47.6" x2="32.5" y2="47" width="0.2" layer="16"/>
+<via x="32.5" y="47" extent="1-16" drill="0.3302"/>
+<wire x1="32.5" y1="47" x2="36.73" y2="47" width="0.2" layer="1"/>
+<wire x1="36.73" y1="47" x2="37.5" y2="47.77" width="0.2" layer="1"/>
 </signal>
 <signal name="VCC">
@@
 <signal name="N$1">
 <contactref element="BUSY" pad="K"/>
-<contactref element="R1" pad="1"/>
-<wire x1="46.5" y1="45.23" x2="46.5" y2="42.95" width="0.2" layer="1"/>
+<contactref element="R1" pad="P$1"/>
+<wire x1="37.5" y1="45.23" x2="38.6621" y2="45.23" width="0.2" layer="1"/>
+<wire x1="38.6621" y1="45.23" x2="39.79605" y2="44.09605" width="0.2" layer="1"/>
 </signal>
 <signal name="N$2">
 <contactref element="ERR" pad="K"/>
-<contactref element="R2" pad="1"/>
-<wire x1="42" y1="45.23" x2="42" y2="42.95" width="0.2" layer="1"/>
+<contactref element="R2" pad="P$1"/>
+<wire x1="41.8" y1="45.23" x2="42.7621" y2="45.23" width="0.2" layer="1"/>
+<wire x1="42.7621" y1="45.23" x2="43.89605" y2="44.09605" width="0.2" layer="1"/>
 </signal>
 <signal name="N$3">
 <contactref element="HI!" pad="K"/>
-<contactref element="R3" pad="1"/>
-<wire x1="37.5" y1="45.23" x2="37.5" y2="42.95" width="0.2" layer="1"/>
+<contactref element="R3" pad="P$1"/>
+<wire x1="46.1" y1="45.23" x2="46.8621" y2="45.23" width="0.2" layer="1"/>
+<wire x1="46.8621" y1="45.23" x2="47.99605" y2="44.09605" width="0.2" layer="1"/>
 </signal>
 <signal name="Z7">
