File: hardware/ziffy_board_v5.sch (EAGLE design)
At the start: 22 parts, among them IC1 ATMEGA328P, Q1 2N3904, Q2 2N3904

Commit message: touch ups, edge routering, etc.
Parts:
- C3: value 0.1uF -> 1uF
Changed lines of the file:
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@@
 <part name="AVR_ISP" library="A_butts" deviceset="AVR_SPI_PRG_6" device="PTH-SHROUD" value="AVR_SPI_PRG_6PTH-SHROUD"/>
 <part name="!HOSTRST" library="A_butts" deviceset="M02" device="PTH"/>
-<part name="C3" library="A_butts" deviceset="CAPACITOR-CERAMIC" device="025-024X044" value="0.1uF"/>
+<part name="C3" library="A_butts" deviceset="CAPACITOR-CERAMIC" device="025-024X044" value="1uF"/>
 <part name="GND1" library="SparkFun-Aesthetics" deviceset="GND" device=""/>
 <part name="SUPPLY4" library="A_butts" deviceset="VCC" device=""/>
